File: bandPass2/bandPass2.kicad_pcb (KiCad board)
At the start: 4 copper layers, 62.5 x 77.2 mm, 114 parts, among them J1 SMA, J11 Conn_01x02, J12 Conn_01x06, J2 SMA, J201 hole, J202 hole, J203 hole, J204 hole, U1 BGS12P2L6E6327XTSA1, U11 BGS12P2L6E6327XTSA1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

Commit message: pcb clean-up
Routing:
- net SEL_BANK2: track 61.3 -> 112.4 mm, vias 2 -> 4
- net GND: vias 22 -> 26
Changed lines of the file:
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@@
   )
   (footprint "Resistor_SMD:R_0805_2012Metric" (layer "F.Cu")
-    (at 101.25 103 -90)
+    (at 101.3 103 -90)
     (descr "Resistor SMD 0805 (2012 Metric), square (rectangular) end terminal, IPC_7351 nominal, (Body size source: IPC-SM-782 page 72, https://www.pcb-3d.com/wordpress/wp-content/uploads/ipc-sm-782a_amendment_1_and_2.pdf), generated with kicad-footprint-generator")
     (tags "resistor")
@@
   (via (at 62.25 88.075) (size 0.8) (drill 0.4) (layers "F.Cu" "B.Cu") (net 2))
   (via (at 56.5 104.5) (size 0.8) (drill 0.4) (layers "F.Cu" "B.Cu") (free) (net 2))
+  (via (at 108 104.5) (size 0.8) (drill 0.4) (layers "F.Cu" "B.Cu") (free) (net 2))
   (via (at 102.25 85.925) (size 0.8) (drill 0.4) (layers "F.Cu" "B.Cu") (net 2))
+  (via (at 109.5 104.5) (size 0.8) (drill 0.4) (layers "F.Cu" "B.Cu") (free) (net 2))
   (via (at 55 95.5) (size 0.8) (drill 0.4) (layers "F.Cu" "B.Cu") (free) (net 2))
   (via (at 62.25 114.075) (size 0.8) (drill 0.4) (layers "F.Cu" "B.Cu") (net 2))
+  (via (at 111 104.5) (size 0.8) (drill 0.4) (layers "F.Cu" "B.Cu") (free) (net 2))
+  (via (at 112.5 104.5) (size 0.8) (drill 0.4) (layers "F.Cu" "B.Cu") (free) (net 2))
   (segment (start 83.25 75.3) (end 83.25 74) (width 1) (layer "B.Cu") (net 3))
   (segment (start 76.7 74) (end 81 74) (width 1) (layer "B.Cu") (net 3))
@@
   (segment (start 73 135.75) (end 73 138.5875) (width 0.5) (layer "B.Cu") (net 29))
   (segment (start 61.8375 97.75) (end 62.6 97.75) (width 0.2) (layer "F.Cu") (net 30))
-  (segment (start 101.25 101.25) (end 101.25 102.0875) (width 0.2) (layer "F.Cu") (net 30))
-  (segment (start 101.3 101.2) (end 101.25 101.25) (width 0.2) (layer "F.Cu") (net 30))
+  (segment (start 101.3 100.4) (end 101.3 102.0875) (width 0.2) (layer "F.Cu") (net 30))
   (segment (start 62.65 98.7) (end 62.6 98.65) (width 0.2) (layer "F.Cu") (net 30))
   (segment (start 63.2 99.25) (end 62.65 98.7) (width 0.2) (layer "F.Cu") (net 30))
+  (segment (start 101.3 102.0875) (end 101.3 102.85) (width 0.2) (layer "F.Cu") (net 30))
   (segment (start 63.2 99.6) (end 63.2 99.25) (width 0.2) (layer "F.Cu") (net 30))
   (segment (start 62.6 98.65) (end 62.6 97.75) (width 0.2) (layer "F.Cu") (net 30))
-  (segment (start 101.25 102.0875) (end 101.25 102.85) (width 0.2) (layer "F.Cu") (net 30))
-  (segment (start 101.3 100.4) (end 101.3 101.2) (width 0.2) (layer "F.Cu") (net 30))
+  (via (at 65.3 93.5) (size 0.8) (drill 0.4) (layers "F.Cu" "B.Cu") (net 30))
   (via (at 62.6 97.75) (size 0.8) (drill 0.4) (layers "F.Cu" "B.Cu") (net 30))
-  (via (at 101.25 102.85) (size 0.8) (drill 0.4) (layers "F.Cu" "B.Cu") (net 30))
+  (via (at 63.2 93.5) (size 0.8) (drill 0.4) (layers "F.Cu" "B.Cu") (net 30))
+  (via (at 101.3 102.85) (size 0.8) (drill 0.4) (layers "F.Cu" "B.Cu") (net 30))
+  (segment (start 65.3 93.5) (end 63.2 93.5) (width 0.5) (layer "In1.Cu") (net 30))
+  (segment (start 101.3 94.8) (end 100 93.5) (width 0.5) (layer "In2.Cu") (net 30))
   (segment (start 60.2 136.9) (end 60.2 100.15) (width 0.5) (layer "In2.Cu") (net 30))
+  (segment (start 62.6 94.1) (end 63.2 93.5) (width 0.5) (layer "In2.Cu") (net 30))
   (segment (start 60.2 100.15) (end 62.6 97.75) (width 0.5) (layer "In2.Cu") (net 30))
   (segment (start 69.7 138.3) (end 61.6 138.3) (width 0.5) (layer "In2.Cu") (net 30))
+  (segment (start 101.3 102.85) (end 101.3 94.8) (width 0.5) (layer "In2.Cu") (net 30))
   (segment (start 61.6 138.3) (end 60.2 136.9) (width 0.5) (layer "In2.Cu") (net 30))
+  (segment (start 62.6 97.75) (end 62.6 94.1) (width 0.5) (layer "In2.Cu") (net 30))
   (segment (start 70.46 135.75) (end 70.46 137.54) (width 0.5) (layer "In2.Cu") (net 30))
   (segment (start 70.46 137.54) (end 69.7 138.3) (width 0.5) (layer "In2.Cu") (net 30))
+  (segment (start 100 93.5) (end 65.3 93.5) (width 0.5) (layer "In2.Cu") (net 30))
   (segment (start 70.46 135.75) (end 70.46 138.5775) (width 0.5) (layer "B.Cu") (net 30))
   (segment (start 70.46 138.5775) (end 70.45 138.5875) (width 0.5) (layer "B.Cu") (net 30))
@@
   (segment (start 61.8375 110.75) (end 62.6 110.75) (width 0.2) (layer "F.Cu") (net 31))
   (via (at 101.3 115.85) (size 0.8) (drill 0.4) (layers "F.Cu" "B.Cu") (net 31))
+  (via (at 65.3 106.5) (size 0.8) (drill 0.4) (layers "F.Cu" "B.Cu") (net 31))
   (via (at 62.6 110.75) (size 0.8) (drill 0.4) (layers "F.Cu" "B.Cu") (net 31))
-  (via (at 63.2 106.4) (size 0.8) (drill 0.4) (layers "F.Cu" "B.Cu") (net 31))
-  (via (at 65.3 106.4) (size 0.8) (drill 0.4) (layers "F.Cu" "B.Cu") (net 31))
-  (segment (start 65.3 106.4) (end 63.2 106.4) (width 0.5) (layer "In1.Cu") (net 31))
-  (segment (start 101.3 115.85) (end 101.3 107.9) (width 0.5) (layer "In2.Cu") (net 31))
+  (via (at 63.2 106.5) (size 0.8) (drill 0.4) (layers "F.Cu" "B.Cu") (net 31))
+  (segment (start 65.3 106.5) (end 63.2 106.5) (width 0.5) (layer "In1.Cu") (net 31))
+  (segment (start 62.6 110.75) (end 62.6 107.1) (width 0.5) (layer "In2.Cu") (net 31))
   (segment (start 62 137.5) (end 61 136.5) (width 0.5) (layer "In2.Cu") (net 31))
-  (segment (start 92.7 106.4) (end 65.3 106.4) (width 0.5) (layer "In2.Cu") (net 31))
-  (segment (start 62.6 107) (end 63.2 106.4) (width 0.5) (layer "In2.Cu") (net 31))
+  (segment (start 101.3 107.8) (end 100 106.5) (width 0.5) (layer "In2.Cu") (net 31))
   (segment (start 61 136.5) (end 61 112.35) (width 0.5) (layer "In2.Cu") (net 31))
+  (segment (start 101.3 115.85) (end 101.3 107.8) (width 0.5) (layer "In2.Cu") (net 31))
   (segment (start 67.3 137.5) (end 62 137.5) (width 0.5) (layer "In2.Cu") (net 31))
-  (segment (start 101.3 107.9) (end 99.9 106.5) (width 0.5) (layer "In2.Cu") (net 31))
-  (segment (start 99.8 106.4) (end 92.7 106.4) (width 0.5) (layer "In2.Cu") (net 31))
+  (segment (start 62.6 107.1) (end 63.2 106.5) (width 0.5) (layer "In2.Cu") (net 31))
   (segment (start 67.92 135.75) (end 67.92 136.88) (width 0.5) (layer "In2.Cu") (net 31))
-  (segment (start 99.9 106.5) (end 99.8 106.4) (width 0.5) (layer "In2.Cu") (net 31))
+  (segment (start 100 106.5) (end 65.3 106.5) (width 0.5) (layer "In2.Cu") (net 31))
   (segment (start 67.92 136.88) (end 67.3 137.5) (width 0.5) (layer "In2.Cu") (net 31))
-  (segment (start 62.6 110.75) (end 62.6 107) (width 0.5) (layer "In2.Cu") (net 31))
   (segment (start 61 112.35) (end 62.6 110.75) (width 0.5) (layer "In2.Cu") (net 31))
   (segment (start 67.92 135.75) (end 67.92 138.5675) (width 0.5) (layer "B.Cu") (net 31))

Commit message: clean-up, add pcb render
Other:
- board text added: "**************** * Max 3.6V * * Unprotected * ****************"
- board text added: "MAX 30dBm UNPROTECTED"
- board text added: "Set HIGH to select"
Changed lines of the file:
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@@
     (property "Sheetname" "")
     (attr through_hole)
-    (fp_text reference "J11" (at 0 -2.33 90) (layer "F.SilkS")
+    (fp_text reference "J11" (at -2.25 0.025 180) (layer "F.SilkS")
       (effects (font (size 0.7 0.7) (thickness 0.1)))
     )
@@
     (effects (font (size 1 1) (thickness 0.15)) (justify right))
   )
+  (gr_text "MAX 30dBm \nUNPROTECTED\n" (at 54.25 111 90) (layer "F.SilkS")
+    (effects (font (size 1 1) (thickness 0.15)))
+  )
   (gr_text "Ch1" (at 72.9 137.5 90) (layer "F.SilkS")
     (effects (font (size 1 1) (thickness 0.15)) (justify right))
@@
     (effects (font (size 1 1) (thickness 0.15)) (justify right))
   )
+  (gr_text "Set HIGH to select" (at 69.2 133.3) (layer "F.SilkS")
+    (effects (font (size 1 1) (thickness 0.15)))
+  )
   (gr_text "Ch0" (at 66.5 69.5) (layer "F.SilkS")
     (effects (font (size 1.5 1.5) (thickness 0.2)))
@@
     (effects (font (size 1 1) (thickness 0.15)) (justify right))
   )
+  (gr_text "MAX 30dBm \nUNPROTECTED\n" (at 110.25 111 270) (layer "F.SilkS")
+    (effects (font (size 1 1) (thickness 0.15)))
+  )
   (gr_text "Ch4" (at 66.5 121.5) (layer "F.SilkS")
     (effects (font (size 1.5 1.5) (thickness 0.2)))
@@
     (effects (font (size 1 1) (thickness 0.15)) (justify right))
   )
+  (gr_text "****************\n* Max 3.6V    *\n* Unprotected *\n****************" (at 88.9 135.8) (layer "F.SilkS")
+    (effects (font (size 1 1) (thickness 0.15)) (justify left))
+  )
   (gr_text "GND" (at 84.5 137.5 90) (layer "F.SilkS")
     (effects (font (size 1 1) (thickness 0.15)) (justify right))
@@
   (segment (start 87.2 126) (end 93.75 126) (width 1) (layer "B.Cu") (net 44))
   (segment (start 63.6625 71.75) (end 65.3625 71.75) (width 0.5) (layer "F.Cu") (net 45))
-  (segment (start 103.425 77.9125) (end 103.45 77.9375) (width 0.5) (layer "F.Cu") (net 46))
-  (segment (start 103.475 77.9125) (end 103.5 77.9375) (width 0.5) (layer "F.Cu") (net 46))
-  (segment (start 101.25 77.9125) (end 103.425 77.9125) (width 0.5) (layer "F.Cu") (net 46))
+  (segment (start 101.3 77.9125) (end 103.425 77.9125) (width 0.5) (layer "F.Cu") (net 46))
   (segment (start 63.6625 84.75) (end 65.3125 84.75) (width 0.5) (layer "F.Cu") (net 47))
-  (segment (start 101.25 90.9125) (end 103.425 90.9125) (width 0.5) (layer "F.Cu") (net 48))
+  (segment (start 101.3 90.9125) (end 103.425 90.9125) (width 0.5) (layer "F.Cu") (net 48))
   (segment (start 103.425 90.9125) (end 103.45 90.9375) (width 0.5) (layer "F.Cu") (net 48))
-  (segment (start 103.475 90.9125) (end 103.5 90.9375) (width 0.5) (layer "F.Cu") (net 48))
   (segment (start 63.6625 97.75) (end 65.3125 97.75) (width 0.5) (layer "F.Cu") (net 49))
-  (segment (start 103.475 103.9125) (end 103.5 103.9375) (width 0.5) (layer "F.Cu") (net 50))
-  (segment (start 103.425 103.9125) (end 103.45 103.9375) (width 0.5) (layer "F.Cu") (net 50))
   (segment (start 101.25 103.9125) (end 103.425 103.9125) (width 0.5) (layer "F.Cu") (net 50))
   (segment (start 63.6625 110.75) (end 65.3125 110.75) (width 0.5) (layer "F.Cu") (net 51))
-  (segment (start 103.425 116.9125) (end 103.45 116.9375) (width 0.5) (layer "F.Cu") (net 52))
   (segment (start 101.3 116.9125) (end 103.425 116.9125) (width 0.5) (layer "F.Cu") (net 52))
-  (segment (start 103.475 116.9125) (end 103.5 116.9375) (width 0.5) (layer "F.Cu") (net 52))
   (segment (start 63.6625 123.75) (end 65.3125 123.75) (width 0.5) (layer "F.Cu") (net 53))
   (segment (start 101.3 129.9125) (end 103.425 129.9125) (width 0.5) (layer "F.Cu") (net 54))
-  (segment (start 103.425 129.9125) (end 103.45 129.9375) (width 0.5) (layer "F.Cu") (net 54))
-  (segment (start 103.475 129.9125) (end 103.5 129.9375) (width 0.5) (layer "F.Cu") (net 54))
   (zone (net 2) (net_name "GND") (layer "F.Cu") (hatch edge 0.508)
     (connect_pads (clearance 0.254))
