File: bandPass2/bandPass2.kicad_pcb (KiCad board)
At the start: 4 copper layers, 62.5 x 77.2 mm, 114 parts, among them J1 SMA, J11 Conn_01x02, J12 Conn_01x06, J2 SMA, J201 hole, J202 hole, J203 hole, J204 hole, U1 BGS12P2L6E6327XTSA1, U11 BGS12P2L6E6327XTSA1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

Commit message: update schematic and pcb
Parts:
- removed D1, D11, D12, D2, D21, D22, D31, D32, D41, D42: KP-2012SURCK, LED_SMD:LED_0805_2012Metric
- removed R10, R11, R12, R13, R14, R15, R6, R7, R8, R9: 1k, Resistor_SMD:R_0805_2012Metric
- removed U1, U2: BGS12P2L6E6327XTSA1, bandPass2:BGS12P2L6E6327XTSA1
- added U01: PE4259, Package_TO_SOT_SMD:SOT-363_SC-70-6, F.Cu at (63.1, 73.3)
- added U02: PE4259, Package_TO_SOT_SMD:SOT-363_SC-70-6, F.Cu at (101.8, 74.7)
- J12: value Conn_01x06 -> Select; footprint Connector_PinHeader_2.54mm:PinHeader_1x06_P2.54mm_Vertical -> Connector_PinHeader_2.54mm:PinHeader_2x05_P2.54mm_Vertical
- R1, R2, R3, R4, R5: moved to F.Cu
- U11, U12, U21, U22, U31, U32, U41, U42: value BGS12P2L6E6327XTSA1 -> PE4259; footprint bandPass2:BGS12P2L6E6327XTSA1 -> Package_TO_SOT_SMD:SOT-363_SC-70-6
- moved R5 71.6 mm to (62.2, 69.2), turned to 90 degrees
- moved R4 60.8 mm to (66.2, 79.1), turned to 0 degrees
- moved R3 47.6 mm to (66.2, 92.1), turned to 0 degrees
- moved R2 34.4 mm to (66.2, 105.1), turned to 0 degrees
- moved R1 21.4 mm to (66.2, 118.1), turned to 0 degrees
- moved C100 1.08 mm to (63.1, 75.9), turned to 180 degrees
- moved C101 1.08 mm to (63.1, 88.9), turned to 180 degrees
- moved C102 1.08 mm to (63.1, 101.9), turned to 180 degrees
- moved C103 1.08 mm to (63.1, 114.9), turned to 180 degrees
- moved C104 1.08 mm to (63.1, 127.9), turned to 180 degrees
- moved C19 0.82 mm to (105.2, 87.7)
- moved C29 0.82 mm to (105.2, 100.7)
- moved C39 0.82 mm to (105.2, 113.7)
- moved C49 0.82 mm to (105.2, 126.7)
- moved C9 0.82 mm to (105.2, 74.7)
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Connections:
- J12 pad 1: SEL_BANK0 -> +3V3
- J12 pad 2: SEL_BANK1 -> SEL_BANK0
- J12 pad 3: SEL_BANK2 -> +3V3
- J12 pad 4: SEL_BANK3 -> SEL_BANK1
- J12 pad 5: SEL_BANK4 -> +3V3
- J12 pad 6: GND -> SEL_BANK2
- U11 pad 1: Net-(C18-Pad2) -> Net-(C11-Pad1)
- U11 pad 3: GND -> unconnected-(U11-Pad3)
- U11 pad 4: +3V3 -> SEL_BANK1
- U11 pad 5: Net-(C11-Pad1) -> Net-(C18-Pad2)
- U11 pad 6: SEL_BANK1 -> +3V3
- U12 pad 1: Net-(C19-Pad1) -> Net-(C17-Pad2)
- U12 pad 3: GND -> unconnected-(U12-Pad3)
- U12 pad 4: +3V3 -> SEL_BANK1
- U12 pad 5: Net-(C17-Pad2) -> Net-(C19-Pad1)
- U12 pad 6: SEL_BANK1 -> +3V3
- U21 pad 1: Net-(C28-Pad2) -> Net-(C21-Pad1)
- U21 pad 3: GND -> unconnected-(U21-Pad3)
- U21 pad 4: +3V3 -> SEL_BANK2
- U21 pad 5: Net-(C21-Pad1) -> Net-(C28-Pad2)
- U21 pad 6: SEL_BANK2 -> +3V3
- U22 pad 1: Net-(C29-Pad1) -> Net-(C27-Pad2)
- U22 pad 3: GND -> unconnected-(U22-Pad3)
- U22 pad 4: +3V3 -> SEL_BANK2
- U22 pad 5: Net-(C27-Pad2) -> Net-(C29-Pad1)
- U22 pad 6: SEL_BANK2 -> +3V3
- U31 pad 1: Net-(C38-Pad2) -> Net-(C31-Pad1)
- U31 pad 3: GND -> unconnected-(U31-Pad3)
- U31 pad 4: +3V3 -> SEL_BANK3
- U31 pad 5: Net-(C31-Pad1) -> Net-(C38-Pad2)
- U31 pad 6: SEL_BANK3 -> +3V3
- U32 pad 1: Net-(C39-Pad1) -> Net-(C37-Pad2)
- U32 pad 3: GND -> unconnected-(U32-Pad3)
- U32 pad 4: +3V3 -> SEL_BANK3
- U32 pad 5: Net-(C37-Pad2) -> Net-(C39-Pad1)
- U32 pad 6: SEL_BANK3 -> +3V3
- U41 pad 1: Net-(C48-Pad2) -> Net-(C41-Pad1)
- U41 pad 3: GND -> unconnected-(U41-Pad3)
- U41 pad 4: +3V3 -> SEL_BANK4
- U41 pad 5: Net-(C41-Pad1) -> Net-(C48-Pad2)
- U41 pad 6: SEL_BANK4 -> +3V3
- U42 pad 1: Net-(C49-Pad1) -> Net-(C47-Pad2)
- U42 pad 3: GND -> unconnected-(U42-Pad3)
- U42 pad 4: +3V3 -> SEL_BANK4
- U42 pad 5: Net-(C47-Pad2) -> Net-(C49-Pad1)
- U42 pad 6: SEL_BANK4 -> +3V3
Routing:
- net GND: track 15.2 -> 0.00 mm, vias 26 -> 96
- net +3V3: track 213.5 -> 205.5 mm
- net SEL_BANK0: track 148.1 -> 144.2 mm
- net SEL_BANK4: track 71.9 -> 74.5 mm
- net Net-(D22-Pad2): track 2.17 -> 0.00 mm
- net Net-(D12-Pad2): track 2.16 -> 0.00 mm
- net Net-(D42-Pad2): track 2.12 -> 0.00 mm
- net Net-(D32-Pad2): track 2.12 -> 0.00 mm
- net Net-(D2-Pad2): track 2.12 -> 0.00 mm
- net Net-(D1-Pad2): track 1.70 -> 0.00 mm
- net SEL_BANK2: track 112.4 -> 110.7 mm
- net Net-(D41-Pad2): track 1.65 -> 0.00 mm
- net Net-(D31-Pad2): track 1.65 -> 0.00 mm
- net Net-(D21-Pad2): track 1.65 -> 0.00 mm
- net Net-(D11-Pad2): track 1.65 -> 0.00 mm
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