File: bandPass2/bandPass2.kicad_sch (KiCad schematic)
At the start: 114 parts, among them J1 SMA, J11 Conn_01x02, J12 Conn_01x06, J2 SMA, J201 hole, J202 hole, J203 hole, J204 hole, U1 BGS12P2L6E6327XTSA1, U11 BGS12P2L6E6327XTSA1, U12 BGS12P2L6E6327XTSA1, U2 BGS12P2L6E6327XTSA1, U21 BGS12P2L6E6327XTSA1, U22 BGS12P2L6E6327XTSA1, U31 BGS12P2L6E6327XTSA1, U32 BGS12P2L6E6327XTSA1, U41 BGS12P2L6E6327XTSA1, U42 BGS12P2L6E6327XTSA1

Commit message: update schematic and pcb
Parts:
- removed D1, D11, D12, D2, D21, D22, D31, D32, D41, D42: KP-2012SURCK, LED_SMD:LED_0805_2012Metric, symbol Device:LED_Small
- removed J12: Conn_01x06, Connector_PinHeader_2.54mm:PinHeader_1x06_P2.54mm_Vertical, symbol Connector_Generic:Conn_01x06
- removed R10, R11, R12, R13, R14, R15, R6, R7, R8, R9: 1k, Resistor_SMD:R_0805_2012Metric, symbol Device:R_Small
- removed U1, U11, U12, U2, U21, U22, U31, U32, U41, U42: BGS12P2L6E6327XTSA1, bandPass2:BGS12P2L6E6327XTSA1, symbol bandPass2:BGS12P2L6E6327XTSA1
- added J12: Select, Connector_PinHeader_2.54mm:PinHeader_2x05_P2.54mm_Vertical, symbol Connector_Generic:Conn_02x05_Odd_Even
- added U01, U02, U11, U12, U21, U22, U31, U32, U41, U42: PE4259, Package_TO_SOT_SMD:SOT-363_SC-70-6, symbol bandPass2:PE4259
Connections:
- net +3V3: now also J12.1 (Pin_1), J12.3 (Pin_3), J12.5 (Pin_5), J12.7 (Pin_7), J12.9 (Pin_9), U01.6 (VDD), U02.6 (VDD), U11.6 (VDD), U12.6 (VDD), U21.6 (VDD), U22.6 (VDD), U31.6 (VDD), U32.6 (VDD), U41.6 (VDD), U42.6 (VDD)
- net GND: now also U01.2 (GND), U02.2 (GND), U11.2 (GND), U12.2 (GND), U21.2 (GND), U22.2 (GND), U31.2 (GND), U32.2 (GND), U41.2 (GND), U42.2 (GND)
- net SEL_BANK0: now also J12.2 (Pin_2), U01.4 (CTRL), U02.4 (CTRL)
- net SEL_BANK1: now also J12.4 (Pin_4), U11.4 (CTRL), U12.4 (CTRL)
- net SEL_BANK2: now also J12.6 (Pin_6), U21.4 (CTRL), U22.4 (CTRL)
- net SEL_BANK3: now also J12.8 (Pin_8), U31.4 (CTRL), U32.4 (CTRL)
- net SEL_BANK4: now also J12.10 (Pin_10), U41.4 (CTRL), U42.4 (CTRL)
- net at C8.2: now also U01.5 (RFIN)
- net at C1.1: now also U01.1 (RF1)
- net at C38.2: now also U31.5 (RFIN)
- net at C31.1: now also U31.1 (RF1)
- net at C37.2: now also U32.1 (RF1)
- net at C21.1: now also U21.1 (RF1)
- net at C28.2: now also U21.5 (RFIN)
- net at C39.1: now also U32.5 (RFIN)
- net at C9.1: now also U02.5 (RFIN)
- net at C17.2: now also U12.1 (RF1)
- net at C48.2: now also U41.5 (RFIN)
- net at C41.1: now also U41.1 (RF1)
- net at C7.2: now also U02.1 (RF1)
- net at C11.1: now also U11.1 (RF1)
- net at C29.1: now also U22.5 (RFIN)
- net at C27.2: now also U22.1 (RF1)
- net at C49.1: now also U42.5 (RFIN)
- net at C47.2: now also U42.1 (RF1)
- net at C18.2: now also U11.5 (RFIN)
- net at C19.1: now also U12.5 (RFIN)
- no-connect marks 0 -> 10
Other:
- note added: "PE4259 truth table ------------------ | CTRL | RF1 | RF2 | ------------------ | 0 | GND | INP | ------------------ | 1 | INP | GND | ------------------"
- moved on the sheet: C1, C100, C101, C102, C103, C104, C105, C106, C107, C108, C109, C11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
